Commit message: Update simple_rocket.urdf

File: simple_rocket.urdf (robot description, URDF)
Before this commit: robot simple_rocket, 2 links, 1 joints
Links:
- removed link body
- removed link nosecone
- added link base_link, mass 10.0; visual cylinder length=0.1524 radius=0.049
- added link engine_link, mass 5.0; visual cylinder length=0.1016 radius=0.049
- added link fins_link, mass 1.0; visual box size=0.0381 0.01905 0.0635
- added link nose_cone_link, mass 2.0; visual cone length=0.0508 radius=0.049
Joints:
- removed joint nosecone_joint
- added joint base_to_engine: type fixed, parent base_link, child engine_link, origin xyz=0.5 0.0 0.0
- added joint base_to_nose_cone: type fixed, parent base_link, child nose_cone_link, origin xyz=0.0 0.0 0.1524
- added joint engine_to_fins: type fixed, parent engine_link, child fins_link, origin xyz=0.0 0.0 -0.25
